File: Hardware/Proiect TSC.brd (EAGLE design)
At the start: 170.2 x 111.2 mm, 103 parts, among them IC1 BD5229G-TR, IC4 XC6220A331MR-G, J1 FH34SRJ-24S-0.5SH_99_, J2 SAMACSYS_PARTS_USB4110-GF-A, J3 QWIIC_RIGHT_ANGLE, J4 112A-TAAR-R03_ATTEND, Q1 20V/4.2A/52mΩ/1.4W, Q2 20V/4.2A/52mΩ/1.4W, Q3 SI1308EDL-T1-GE3, U1 W25Q512JVEIQ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

Commit message: Fixes #1 #2 #3 #4 #5 #6 #7 #8 #9
Parts:
- R1, R_CHANGE: value (none) -> 10K
Connections:
- removed net N$16: EPD_C11.1, J1.23
- removed net N$7: D5.1
- net PREVGH: now also D5.1, EPD_C9.1, J1.21; no longer D4.2
- net PREVGL: now also D4.2, EPD_C11.1, J1.23; no longer EPD_C9.1, J1.21
Routing:
- net PREVGL: track 9.42 -> 39.3 mm, vias 2 -> 5
- net PREVGH: track 0.00 -> 29.4 mm, vias 0 -> 4
- net N$16: track 22.1 -> 0.00 mm, vias 4 -> 0
- net 3V3: track 440.2 -> 443.6 mm
- net GND: track 665.6 -> 667.0 mm
- net VBUS: track 98.8 -> 99.5 mm
- net MISO: track 103.8 -> 104.4 mm
Other:
- board text added: "3V3"
- board text added: "EPD_3V3_C"
- board text added: "EPD_BUSY"
- board text added: "EPD_CS"
- board text added: "EPD_DC"
- board text added: "EPD_RS"
- board text added: "GND"
- board text added: "INT_RTC"
- board text added: "MISO"
- board text added: "MOSI"
- board text added: "RX"
- board text added: "SCK"
- board text added: "TX"
- board text added: "VBAT"
- board text added: "VBUS"
