File: Hardware/Proiect TSC.sch (EAGLE design)
At the start: 103 parts, among them IC1 BD5229G-TR, IC4 XC6220A331MR-G, J1 FH34SRJ-24S-0.5SH_99_, J2 SAMACSYS_PARTS_USB4110-GF-A, J3 QWIIC_RIGHT_ANGLE, J4 112A-TAAR-R03_ATTEND, Q1 20V/4.2A/52mΩ/1.4W, Q2 20V/4.2A/52mΩ/1.4W, Q3 SI1308EDL-T1-GE3, U1 W25Q512JVEIQ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

Commit message: Fixes #1 #2 #3 #4 #5 #6 #7 #8 #9
Parts:
- R1, R_CHANGE: value (none) -> 10K
Connections:
- removed net N$16: EPD_C11.1, J1.23
- removed net N$7: D5.K
- net PREVGH: now also D5.K, EPD_C9.1, J1.21; no longer D4.A
- net PREVGL: now also D4.A, EPD_C11.1, J1.23; no longer EPD_C9.1, J1.21
Other:
- moved on the sheet: EPD_C10
Changed lines of the file:
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@@
 </classes>
 <parts>
-<part name="FRAME1" library="DeskAssistant v19 v1" library_urn="urn:adsk.wipprod:fs.file:vf.6UOSBqwYQ-e5e-3uXwhMQA" deviceset="ESP32_WROVER_FRAMES_A3L-LOC" device=""/>
+<part name="FRAME1" library="DeskAssistant v19 v1" library_urn="urn:adsk.wipprod:fs.file:vf.6UOSBqwYQ-e5e-3uXwhMQA" deviceset="ESP32_WROVER_FRAMES_A3L-LOC" device="" value="SCHEMATIC"/>
 <part name="J2" library="DeskAssistant v19 v1" library_urn="urn:adsk.wipprod:fs.file:vf.6UOSBqwYQ-e5e-3uXwhMQA" deviceset="SAMACSYS_PARTS_USB4110-GF-A" device="" value="SAMACSYS_PARTS_USB4110-GF-A"/>
 <part name="PFMF.050.1" library="DeskAssistant v19 v1" library_urn="urn:adsk.wipprod:fs.file:vf.6UOSBqwYQ-e5e-3uXwhMQA" deviceset="ESP32C6_VARISTOR" device="CN1812" value="ESP32C6_VARISTORCN1812"/>
@@
 <part name="C2_BAT" library="DeskAssistant v19 v1" library_urn="urn:adsk.wipprod:fs.file:vf.6UOSBqwYQ-e5e-3uXwhMQA" deviceset="EAGLE-LTSPICE_C" device="C0402" value="4.7uF"/>
 <part name="U2" library="DeskAssistant v19 v1" library_urn="urn:adsk.wipprod:fs.file:vf.6UOSBqwYQ-e5e-3uXwhMQA" deviceset="ESP32-C6-WROOM-1-N8" device=""/>
-<part name="R1" library="DeskAssistant v19 v1" library_urn="urn:adsk.wipprod:fs.file:vf.6UOSBqwYQ-e5e-3uXwhMQA" deviceset="ESP32_WROVER_EAGLE-LTSPICE_R" device="R0402"/>
+<part name="R1" library="DeskAssistant v19 v1" library_urn="urn:adsk.wipprod:fs.file:vf.6UOSBqwYQ-e5e-3uXwhMQA" deviceset="ESP32_WROVER_EAGLE-LTSPICE_R" device="R0402" value="10K"/>
 <part name="SUPPLY24" library="DeskAssistant v19 v1" library_urn="urn:adsk.wipprod:fs.file:vf.6UOSBqwYQ-e5e-3uXwhMQA" deviceset="GND-BAR" device="" value="GND"/>
 <part name="SUPPLY25" library="DeskAssistant v19 v1" library_urn="urn:adsk.wipprod:fs.file:vf.6UOSBqwYQ-e5e-3uXwhMQA" deviceset="3V3-CIRCLE" device="" value="3V3"/>
@@
 <part name="SUPPLY40" library="DeskAssistant v19 v1" library_urn="urn:adsk.wipprod:fs.file:vf.6UOSBqwYQ-e5e-3uXwhMQA" deviceset="GND-BAR" device="" value="GND"/>
 <part name="R_BOOT" library="DeskAssistant v19 v1" library_urn="urn:adsk.wipprod:fs.file:vf.6UOSBqwYQ-e5e-3uXwhMQA" deviceset="ESP32_WROVER_EAGLE-LTSPICE_R" device="R0402" value="10K"/>
-<part name="R_CHANGE" library="DeskAssistant v19 v1" library_urn="urn:adsk.wipprod:fs.file:vf.6UOSBqwYQ-e5e-3uXwhMQA" deviceset="ESP32_WROVER_EAGLE-LTSPICE_R" device="R0402"/>
+<part name="R_CHANGE" library="DeskAssistant v19 v1" library_urn="urn:adsk.wipprod:fs.file:vf.6UOSBqwYQ-e5e-3uXwhMQA" deviceset="ESP32_WROVER_EAGLE-LTSPICE_R" device="R0402" value="10K"/>
 <part name="BOOT_BUTTON" library="DeskAssistant v19 v1" library_urn="urn:adsk.wipprod:fs.file:vf.6UOSBqwYQ-e5e-3uXwhMQA" deviceset="BUTTON_CUSYOMV1" device="" value="BUTTON_CUSYOMV1"/>
 <part name="CHANGE_BUTTON" library="DeskAssistant v19 v1" library_urn="urn:adsk.wipprod:fs.file:vf.6UOSBqwYQ-e5e-3uXwhMQA" deviceset="BUTTON_CUSYOMV1" device="" value="BUTTON_CUSYOMV1"/>
@@
 <attribute name="VALUE" x="16.764" y="132.461" size="1.778" layer="96"/>
 </instance>
-<instance part="EPD_C10" gate="G$1" x="38.1" y="132.08" smashed="yes" rot="R270">
-<attribute name="NAME" x="24.384" y="129.921" size="1.778" layer="95"/>
-<attribute name="VALUE" x="39.624" y="129.921" size="1.778" layer="96"/>
+<instance part="EPD_C10" gate="G$1" x="40.64" y="132.08" smashed="yes" rot="R270">
+<attribute name="NAME" x="26.924" y="129.921" size="1.778" layer="95"/>
+<attribute name="VALUE" x="42.164" y="129.921" size="1.778" layer="96"/>
 </instance>
 <instance part="EPD_C9" gate="G$1" x="22.86" y="129.54" smashed="yes" rot="R270">
@@
 <wire x1="22.86" y1="134.62" x2="7.62" y2="134.62" width="0.1524" layer="91"/>
 <wire x1="7.62" y1="134.62" x2="7.62" y2="137.16" width="0.1524" layer="91"/>
-<junction x="7.62" y="137.16"/>
-<wire x1="33.02" y1="132.08" x2="7.62" y2="132.08" width="0.1524" layer="91"/>
+<wire x1="35.56" y1="132.08" x2="7.62" y2="132.08" width="0.1524" layer="91"/>
 <wire x1="7.62" y1="132.08" x2="7.62" y2="134.62" width="0.1524" layer="91"/>
-<junction x="7.62" y="134.62"/>
 <wire x1="17.78" y1="129.54" x2="7.62" y2="129.54" width="0.1524" layer="91"/>
 <wire x1="7.62" y1="129.54" x2="7.62" y2="132.08" width="0.1524" layer="91"/>
-<junction x="7.62" y="132.08"/>
 <wire x1="27.94" y1="127" x2="7.62" y2="127" width="0.1524" layer="91"/>
 <wire x1="7.62" y1="127" x2="7.62" y2="129.54" width="0.1524" layer="91"/>
-<junction x="7.62" y="129.54"/>
 <wire x1="17.78" y1="124.46" x2="7.62" y2="124.46" width="0.1524" layer="91"/>
 <wire x1="7.62" y1="124.46" x2="7.62" y2="127" width="0.1524" layer="91"/>
-<junction x="7.62" y="127"/>
 <wire x1="27.94" y1="121.92" x2="7.62" y2="121.92" width="0.1524" layer="91"/>
 <wire x1="7.62" y1="121.92" x2="7.62" y2="124.46" width="0.1524" layer="91"/>
-<junction x="7.62" y="124.46"/>
 <wire x1="10.16" y1="114.3" x2="7.62" y2="114.3" width="0.1524" layer="91"/>
 <wire x1="7.62" y1="114.3" x2="7.62" y2="121.92" width="0.1524" layer="91"/>
-<junction x="7.62" y="121.92"/>
 <pinref part="EPD_C12" gate="G$1" pin="2"/>
 <pinref part="EPD_C11" gate="G$1" pin="2"/>
@@
 <pinref part="EPD_C6" gate="G$1" pin="2"/>
 <pinref part="EPD_C5" gate="G$1" pin="2"/>
+<junction x="7.62" y="137.16"/>
+<junction x="7.62" y="134.62"/>
+<junction x="7.62" y="132.08"/>
+<junction x="7.62" y="129.54"/>
+<junction x="7.62" y="127"/>
+<junction x="7.62" y="124.46"/>
+<junction x="7.62" y="121.92"/>
 </segment>
 <segment>
@@
 <net name="PREVGH" class="0">
 <segment>
-<wire x1="104.14" y1="177.8" x2="106.68" y2="177.8" width="0.1524" layer="91"/>
-<label x="106.68" y="177.8" size="1.27" layer="95" xref="yes"/>
+<wire x1="45.72" y1="129.54" x2="33.02" y2="129.54" width="0.1524" layer="91"/>
+<label x="33.02" y="139.7" size="1.27" layer="95" rot="R90" xref="yes"/>
+<wire x1="33.02" y1="129.54" x2="25.4" y2="129.54" width="0.1524" layer="91"/>
+<wire x1="33.02" y1="129.54" x2="33.02" y2="139.7" width="0.1524" layer="91"/>
+<pinref part="EPD_C9" gate="G$1" pin="1"/>
+<pinref part="J1" gate="G$1" pin="21"/>
+<junction x="33.02" y="129.54"/>
+</segment>
+<segment>
+<wire x1="106.68" y1="165.1" x2="104.14" y2="165.1" width="0.1524" layer="91"/>
+<pinref part="D5" gate="G$1" pin="K"/>
 <label x="106.68" y="165.1" size="1.27" layer="95" xref="yes"/>
-<pinref part="D4" gate="G$1" pin="A"/>
-</segment>
-</net>
-<net name="N$7" class="0">
-<segment>
-<wire x1="104.14" y1="165.1" x2="106.68" y2="165.1" width="0.1524" layer="91"/>
-<pinref part="D5" gate="G$1" pin="K"/>
 </segment>
 </net>
@@
 <net name="PREVGL" class="0">
 <segment>
-<wire x1="45.72" y1="129.54" x2="30.48" y2="129.54" width="0.1524" layer="91"/>
-<label x="30.48" y="139.7" size="1.27" layer="95" rot="R90" xref="yes"/>
-<wire x1="30.48" y1="129.54" x2="25.4" y2="129.54" width="0.1524" layer="91"/>
-<junction x="30.48" y="129.54"/>
-<wire x1="30.48" y1="129.54" x2="30.48" y2="139.7" width="0.1524" layer="91"/>
-<pinref part="EPD_C9" gate="G$1" pin="1"/>
-<pinref part="J1" gate="G$1" pin="21"/>
+<wire x1="45.72" y1="134.62" x2="38.1" y2="134.62" width="0.1524" layer="91"/>
+<wire x1="38.1" y1="134.62" x2="38.1" y2="139.7" width="0.1524" layer="91"/>
+<label x="38.1" y="139.7" size="1.27" layer="95" rot="R90" xref="yes"/>
+<wire x1="38.1" y1="134.62" x2="30.48" y2="134.62" width="0.1524" layer="91"/>
+<pinref part="EPD_C11" gate="G$1" pin="1"/>
+<pinref part="J1" gate="G$1" pin="23"/>
+<junction x="38.1" y="134.62"/>
+</segment>
+<segment>
+<wire x1="104.14" y1="177.8" x2="106.68" y2="177.8" width="0.1524" layer="91"/>
+<label x="106.68" y="177.8" size="1.27" layer="95" xref="yes"/>
+<pinref part="D4" gate="G$1" pin="A"/>
 </segment>
 </net>
 <net name="N$10" class="0">
 <segment>
-<wire x1="45.72" y1="132.08" x2="40.64" y2="132.08" width="0.1524" layer="91"/>
+<wire x1="45.72" y1="132.08" x2="43.18" y2="132.08" width="0.1524" layer="91"/>
 <pinref part="EPD_C10" gate="G$1" pin="1"/>
 <pinref part="J1" gate="G$1" pin="22"/>
@@
 </segment>
 </net>
-<net name="N$16" class="0">
-<segment>
-<wire x1="45.72" y1="134.62" x2="38.1" y2="134.62" width="0.1524" layer="91"/>
-<wire x1="38.1" y1="134.62" x2="38.1" y2="139.7" width="0.1524" layer="91"/>
-<label x="38.1" y="139.7" size="1.27" layer="95" rot="R90" xref="yes"/>
-<wire x1="38.1" y1="134.62" x2="30.48" y2="134.62" width="0.1524" layer="91"/>
-<junction x="38.1" y="134.62"/>
-<pinref part="EPD_C11" gate="G$1" pin="1"/>
-<pinref part="J1" gate="G$1" pin="23"/>
-</segment>
-</net>
